Commit message: experimenting with gazebo and inertial features

File: src/my_robot_description/urdf/common_properties.xacro (robot description, xacro)
@@ -10,3 +10,12 @@
         <color rgba="0 0 0.7 1"/>
     </material>
+    <xacro:macro name="box_inertia" params="m x y z o_xyz o_rpy">
+    <inertial>
+        <origin xyz="${o_xyz}" rpy="${o_rpy}"/>
+        <mass value="${m}"/>
+        <inertia ixx="${m*(y*y + z*z)/12}" ixy="0" ixz="0"
+                 iyy="${m*(x*x + z*z)/12}" iyz="0"
+                 izz="${m*(y*y + x*x)/12}"/>
+    </inertial>
+    </xacro:macro>
 </robot>

File: src/my_robot_description/urdf/mobile_base.xacro (robot description, xacro)
@@ -20,4 +20,5 @@
             <material name="green"/>
         </visual>
+        <xacro:box_inertia m="5.0" x="${base_length}" y="${base_width}" z="${base_height}" o_xyz="0 0 ${base_height/2.0}" o_rpy="0 0 0" />
     </link>
     <link name="second_link">

Commit message: Working with Macros and Gazebo

File: src/my_robot_description/urdf/common_properties.xacro (robot description, xacro)
@@ -19,3 +19,21 @@
     </inertial>
     </xacro:macro>
+    <xacro:macro name="cylinderical_inertia" params="m r l o_xyz o_rpy">
+    <inertial>
+        <origin xyz="${o_xyz}" rpy="${o_rpy}"/>
+        <mass value="${m}"/>
+        <inertia ixx="${m*(3*r*r + l*l)/12}" ixy="0" ixz="0"
+                 iyy="${m*(3*r*r + l*l)/12}" iyz="0"
+                 izz="${m*(r*r)/2}"/>
+    </inertial>
+    </xacro:macro>
+    <xacro:macro name="spherical_inertia" params="m r  o_xyz o_rpy">
+    <inertial>
+        <origin xyz="${o_xyz}" rpy="${o_rpy}"/>
+        <mass value="${m}"/>
+        <inertia ixx="${m*(2*r*r)/3}" ixy="0" ixz="0"
+                 iyy="${m*(2*r*r)/3}" iyz="0"
+                 izz="${m*(2*r*r)/3}"/>
+    </inertial>
+    </xacro:macro>
 </robot>

File: src/my_robot_description/urdf/mobile_base.xacro (robot description, xacro)
@@ -20,4 +20,10 @@
             <material name="green"/>
         </visual>
+        <collision>
+            <geometry>
+                <box size="${base_length} ${base_width} ${base_height}" />
+            </geometry>
+            <origin xyz="0 0 ${base_height/2.0}" rpy="0 0 0" />
+        </collision>
         <xacro:box_inertia m="5.0" x="${base_length}" y="${base_width}" z="${base_height}" o_xyz="0 0 ${base_height/2.0}" o_rpy="0 0 0" />
     </link>
@@ -30,4 +36,11 @@
             <material name="grey"/>
         </visual>
+        <collision>
+            <geometry>
+                <cylinder radius="${sholder_radius}" length="${sholder_length}"/>
+            </geometry>
+            <origin xyz="0 0 ${base_height/2.0}" rpy="0 0 0" />
+        </collision>
+        <xacro:cylinderical_inertia m="0.6545" r="${sholder_radius}" l="${sholder_length}" o_xyz="0 0 ${base_height/2.0}" o_rpy="0 0 0" />
     </link>
     <link name="third_link">
@@ -39,4 +52,11 @@
             <material name="blue"/>
         </visual>
+        <collision>
+            <geometry>
+                <box size="${claw_length} ${claw_width} ${claw_height}"/>
+            </geometry>
+            <origin xyz="0 ${claw_width/2.0} ${claw_height/2.0}" rpy="0 0 0" />
+        </collision>
+        <xacro:box_inertia m="0.02604" x="${claw_length}" y="${claw_width}" z="${claw_height}" o_xyz=" 0 ${claw_width/2.0} ${claw_height/2.0}" o_rpy="0 0 0" />
     </link>
     <link name="forth_link">
@@ -48,4 +68,11 @@
             <material name="blue"/>
         </visual>
+        <collision>
+            <geometry>
+                <box size="${claw_length} ${claw_width} ${claw_height}"/>
+            </geometry>
+            <origin xyz="0 ${-claw_width/2.0} ${claw_height/2.0}" rpy="0 0 0" />
+        </collision>
+        <xacro:box_inertia m="0.02604" x="${claw_length}" y="${claw_width}" z="${claw_height}" o_xyz="0 ${-claw_width/2.0} ${claw_height/2.0}" o_rpy="0 0 0" />
     </link>
     <!-- <link name="right_front_wheel">
@@ -76,4 +103,11 @@
                 <material name="blue"/>
             </visual>
+            <collision>
+                <geometry>
+                    <sphere radius="${wheel_radius}" />
+                </geometry>
+                <origin xyz="0 ${y*wheel_length/2.0} 0" rpy="0 0 0" />
+            </collision>
+            <xacro:cylinderical_inertia m="1" r="${wheel_radius}" l="${wheel_length}" o_xyz="0 ${y*wheel_length/2.0} 0" o_rpy="${pi/2.0} 0 0" />
         </link>
     </xacro:macro>
@@ -106,4 +140,11 @@
             <material name="blue"/>
         </visual>
+        <collision>
+            <geometry>
+                <sphere radius="${caster_wheel_radius}"/>
+            </geometry>
+            <origin xyz="0 0 0" rpy="0 0 0" />
+        </collision>
+        <xacro:spherical_inertia m="0.5" r="${caster_wheel_radius}" o_xyz="0 0 0" o_rpy="0 0 0"/>
     </link>
     <link name="base_footprint">
@@ -162,5 +203,5 @@
         <parent link="base_footprint" />
         <child link="base_link" />
-        <origin xyz="0 0 0.1" rpy="0 0 0"/>
+        <origin xyz="0 0 ${wheel_radius}" rpy="0 0 0"/>
     </joint>
 </robot>

Commit message: Working on ROS-Gazebo Bridge Node

File: src/my_robot_description/urdf/common_properties.xacro (robot description, xacro)
@@ -34,5 +34,5 @@
         <inertia ixx="${m*(2*r*r)/3}" ixy="0" ixz="0"
                  iyy="${m*(2*r*r)/3}" iyz="0"
-                 izz="${m*(2*r*r)/3}"/>
+                 izz="${m*(r*r)/2}"/>
     </inertial>
     </xacro:macro>

File: src/my_robot_description/urdf/mobile_base.xacro (robot description, xacro)
@@ -6,9 +6,4 @@
     <xacro:property name="wheel_radius" value="0.2"/>
     <xacro:property name="wheel_length" value="0.1"/>
-    <xacro:property name="sholder_radius" value="0.2"/>
-    <xacro:property name="sholder_length" value="0.4"/>
-    <xacro:property name="claw_length" value="0.2"/>
-    <xacro:property name="claw_width" value="0.1"/>
-    <xacro:property name="claw_height" value="0.2"/>
     <xacro:property name="caster_wheel_radius" value="0.1"/>
     <link name="base_link">
@@ -28,70 +23,4 @@
         <xacro:box_inertia m="5.0" x="${base_length}" y="${base_width}" z="${base_height}" o_xyz="0 0 ${base_height/2.0}" o_rpy="0 0 0" />
     </link>
-    <link name="second_link">
-        <visual>
-            <geometry>
-                <cylinder radius="${sholder_radius}" length="${sholder_length}"/>
-            </geometry>
-            <origin xyz="0 0 ${base_height/2.0}" rpy="0 0 0" />
-            <material name="grey"/>
-        </visual>
-        <collision>
-            <geometry>
-                <cylinder radius="${sholder_radius}" length="${sholder_length}"/>
-            </geometry>
-            <origin xyz="0 0 ${base_height/2.0}" rpy="0 0 0" />
-        </collision>
-        <xacro:cylinderical_inertia m="0.6545" r="${sholder_radius}" l="${sholder_length}" o_xyz="0 0 ${base_height/2.0}" o_rpy="0 0 0" />
-    </link>
-    <link name="third_link">
-        <visual>
-            <geometry>
-                <box size="${claw_length} ${claw_width} ${claw_height}"/>
-            </geometry>
-            <origin xyz="0 ${claw_width/2.0} ${claw_height/2.0}" rpy="0 0 0" />
-            <material name="blue"/>
-        </visual>
-        <collision>
-            <geometry>
-                <box size="${claw_length} ${claw_width} ${claw_height}"/>
-            </geometry>
-            <origin xyz="0 ${claw_width/2.0} ${claw_height/2.0}" rpy="0 0 0" />
-        </collision>
-        <xacro:box_inertia m="0.02604" x="${claw_length}" y="${claw_width}" z="${claw_height}" o_xyz=" 0 ${claw_width/2.0} ${claw_height/2.0}" o_rpy="0 0 0" />
-    </link>
-    <link name="forth_link">
-        <visual>
-            <geometry>
-                <box size="${claw_length} ${claw_width} ${claw_height}"/>
-            </geometry>
-            <origin xyz="0 ${-claw_width/2.0} ${claw_height/2.0}" rpy="0 0 0" />
-            <material name="blue"/>
-        </visual>
-        <collision>
-            <geometry>
-                <box size="${claw_length} ${claw_width} ${claw_height}"/>
-            </geometry>
-            <origin xyz="0 ${-claw_width/2.0} ${claw_height/2.0}" rpy="0 0 0" />
-        </collision>
-        <xacro:box_inertia m="0.02604" x="${claw_length}" y="${claw_width}" z="${claw_height}" o_xyz="0 ${-claw_width/2.0} ${claw_height/2.0}" o_rpy="0 0 0" />
-    </link>
-    <!-- <link name="right_front_wheel">
-        <visual>
-            <geometry>
-                <cylinder radius="0.1" length="0.05"/>
-            </geometry>
-            <origin xyz="0 0.025 0" rpy="1.57 0 0" />
-            <material name="blue"/>
-        </visual>
-    </link>
-    <link name="left_front_wheel">
-        <visual>
-            <geometry>
-                <cylinder radius="0.1" length="0.05"/>
-            </geometry>
-            <origin xyz="0 -0.025 0" rpy="1.57 0 0" />
-            <material name="blue"/>
-        </visual>
-    </link> -->
     <xacro:macro name="wheel" params="prefix y">
         <link name="${prefix}_wheel">
@@ -114,22 +43,4 @@
     <xacro:wheel prefix="right" y="1" />
     <xacro:wheel prefix="left"  y="-1"/>
-    <!-- <link name="left_rear_wheel">
-        <visual>
-            <geometry>
-                <cylinder radius="${wheel_radius}" length="${wheel_length}"/>
-            </geometry>
-            <origin xyz="0 ${-wheel_length/2.0} 0" rpy="${pi/2.0} 0 0" />
-            <material name="blue"/>
-        </visual>
-    </link>
-    <link name="right_rear_wheel">
-        <visual>
-            <geometry>
-                <cylinder radius="${wheel_radius}" length="${wheel_length}"/>
-            </geometry>
-            <origin xyz="0 ${wheel_length/2.0} 0" rpy="${pi/2.0} 0 0" />
-            <material name="blue"/>
-        </visual>
-    </link> -->
     <link name="caster_wheel_link">
         <visual>
@@ -150,37 +61,4 @@
     <link name="base_footprint">
     </link>
-     <joint name="base_second_joint" type="continuous">
-        <parent link="base_link" />
-        <child link="second_link" />
-        <axis xyz="0 0 1" />
-        <!-- <limit lower="1.57" upper="-1.57" velocity ="100" effort="100" /> -->
-        <origin xyz="0 0 ${base_height}" rpy="0 0 0"/>
-    </joint>
-    <joint name="second_third_joint" type="prismatic">
-        <parent link="second_link" />
-        <child link="third_link" />
-        <origin xyz="0 0 ${sholder_length}" rpy="0 0 0"/>
-        <axis xyz="0 1 0"/>
-        <limit lower="0.0" upper="0.025" velocity ="100" effort="100"/>
-    </joint>
-    <joint name="second_forth_joint" type="prismatic">
-        <parent link="second_link" />
-        <child link="forth_link" />
-        <origin xyz="0 0 ${sholder_length}" rpy="0 0 0"/>
-        <axis xyz="0 1 0"/>
-        <limit lower="-0.025" upper="0" velocity ="100" effort="100"/>
-    </joint>
-    <!-- <joint name="Base_right_f_wheel" type="continuous">
-        <parent link="base_link" />
-        <child link="right_front_wheel" />
-        <origin xyz="0.25 0.2 0" rpy="0 0 0"/>
-        <axis xyz="0 1 0"/>
-    </joint>
-    <joint name="Base_left_f_wheel" type="continuous">
-        <parent link="base_link" />
-        <child link="left_front_wheel" />
-        <origin xyz="0.25 -0.2 0" rpy="0 0 0"/>
-        <axis xyz="0 1 0"/>
-    </joint> -->
     <joint name="Base_left_r_wheel" type="continuous">
         <parent link="base_link" />

File: src/my_robot_description/urdf/my_robot.urdf.xacro (robot description, xacro)
@@ -3,3 +3,4 @@
     <xacro:include filename="common_properties.xacro"/>
     <xacro:include filename="mobile_base.xacro"/>
+    <xacro:include filename="mobile_base_gazebo.xacro"/>
 </robot>
