Commit message: Learnt and Implimented Xacro in the URDF

File: src/my_robot_description/urdf/mobile_base.xacro (robot description, xacro)
@@ -1,19 +1,21 @@
 <?xml version="1.0"?>
-<robot name="my_robot">
-    <material name="green">
-        <color rgba="0 0.5 0 1"/>
-    </material>
-    <material name="grey">
-        <color rgba="0.5 0.5 0.5 1"/>
-    </material>
-    <material name="blue">
-        <color rgba="0 0 0.7 1"/>
-    </material>
+<robot xmlns:xacro="http://www.ros.org/wiki/xacro">
+    <xacro:property name="base_length" value="1.2"/>
+    <xacro:property name="base_width" value="0.8"/>
+    <xacro:property name="base_height" value="0.4"/>
+    <xacro:property name="wheel_radius" value="0.2"/>
+    <xacro:property name="wheel_length" value="0.1"/>
+    <xacro:property name="sholder_radius" value="0.2"/>
+    <xacro:property name="sholder_length" value="0.4"/>
+    <xacro:property name="claw_length" value="0.2"/>
+    <xacro:property name="claw_width" value="0.1"/>
+    <xacro:property name="claw_height" value="0.2"/>
+    <xacro:property name="caster_wheel_radius" value="0.1"/>
     <link name="base_link">
         <visual>
             <geometry>
-                <box size="0.6 0.4 0.2" />
+                <box size="${base_length} ${base_width} ${base_height}" />
             </geometry>
-            <origin xyz="0 0 0.1" rpy="0 0 0" />
+            <origin xyz="0 0 ${base_height/2.0}" rpy="0 0 0" />
             <material name="green"/>
         </visual>
@@ -22,7 +24,7 @@
         <visual>
             <geometry>
-                <cylinder radius="0.1" length="0.2"/>
+                <cylinder radius="${sholder_radius}" length="${sholder_length}"/>
             </geometry>
-            <origin xyz="0 0 0.1" rpy="0 0 0" />
+            <origin xyz="0 0 ${base_height/2.0}" rpy="0 0 0" />
             <material name="grey"/>
         </visual>
@@ -31,7 +33,7 @@
         <visual>
             <geometry>
-                <box size="0.1 0.05 0.1"/>
+                <box size="${claw_length} ${claw_width} ${claw_height}"/>
             </geometry>
-            <origin xyz="0 0.025 0.05" rpy="0 0 0" />
+            <origin xyz="0 ${claw_width/2.0} ${claw_height/2.0}" rpy="0 0 0" />
             <material name="blue"/>
         </visual>
@@ -40,7 +42,7 @@
         <visual>
             <geometry>
-                <box size="0.1 0.05 0.1"/>
+                <box size="${claw_length} ${claw_width} ${claw_height}"/>
             </geometry>
-            <origin xyz="0 -0.025 0.05" rpy="0 0 0" />
+            <origin xyz="0 ${-claw_width/2.0} ${claw_height/2.0}" rpy="0 0 0" />
             <material name="blue"/>
         </visual>
@@ -64,10 +66,23 @@
         </visual>
     </link> -->
-    <link name="left_rear_wheel">
+    <xacro:macro name="wheel" params="prefix y">
+        <link name="${prefix}_wheel">
+            <visual>
+                <geometry>
+                    <cylinder radius="${wheel_radius}" length="${wheel_length}"/>
+                </geometry>
+                <origin xyz="0 ${y*wheel_length/2.0} 0" rpy="${pi/2.0} 0 0" />
+                <material name="blue"/>
+            </visual>
+        </link>
+    </xacro:macro>
+    <xacro:wheel prefix="right" y="1" />
+    <xacro:wheel prefix="left"  y="-1"/>
+    <!-- <link name="left_rear_wheel">
         <visual>
             <geometry>
-                <cylinder radius="0.1" length="0.05"/>
+                <cylinder radius="${wheel_radius}" length="${wheel_length}"/>
             </geometry>
-            <origin xyz="0 -0.025 0" rpy="1.57 0 0" />
+            <origin xyz="0 ${-wheel_length/2.0} 0" rpy="${pi/2.0} 0 0" />
             <material name="blue"/>
         </visual>
@@ -76,14 +91,14 @@
         <visual>
             <geometry>
-                <cylinder radius="0.1" length="0.05"/>
+                <cylinder radius="${wheel_radius}" length="${wheel_length}"/>
             </geometry>
-            <origin xyz="0 0.025 0" rpy="1.57 0 0" />
+            <origin xyz="0 ${wheel_length/2.0} 0" rpy="${pi/2.0} 0 0" />
             <material name="blue"/>
         </visual>
-    </link>
+    </link> -->
     <link name="caster_wheel_link">
         <visual>
             <geometry>
-                <sphere radius="0.05"/>
+                <sphere radius="${caster_wheel_radius}"/>
             </geometry>
             <origin xyz="0 0 0" rpy="0 0 0" />
@@ -98,10 +113,10 @@
         <axis xyz="0 0 1" />
         <!-- <limit lower="1.57" upper="-1.57" velocity ="100" effort="100" /> -->
-        <origin xyz="0 0 0.2" rpy="0 0 0"/>
+        <origin xyz="0 0 ${base_height}" rpy="0 0 0"/>
     </joint>
     <joint name="second_third_joint" type="prismatic">
         <parent link="second_link" />
         <child link="third_link" />
-        <origin xyz="0 0 0.2" rpy="0 0 0"/>
+        <origin xyz="0 0 ${sholder_length}" rpy="0 0 0"/>
         <axis xyz="0 1 0"/>
         <limit lower="0.0" upper="0.025" velocity ="100" effort="100"/>
@@ -110,5 +125,5 @@
         <parent link="second_link" />
         <child link="forth_link" />
-        <origin xyz="0 0 0.2" rpy="0 0 0"/>
+        <origin xyz="0 0 ${sholder_length}" rpy="0 0 0"/>
         <axis xyz="0 1 0"/>
         <limit lower="-0.025" upper="0" velocity ="100" effort="100"/>
@@ -128,12 +143,12 @@
     <joint name="Base_left_r_wheel" type="continuous">
         <parent link="base_link" />
-        <child link="left_rear_wheel" />
-        <origin xyz="-0.25 -0.2 0" rpy="0 0 0"/>
+        <child link="left_wheel" />
+        <origin xyz="${-((base_length/2.0)-0.05)} ${-base_width/2.0} 0" rpy="0 0 0"/>
         <axis xyz="0 1 0"/>
     </joint>
     <joint name="Base_right_r_wheel" type="continuous">
         <parent link="base_link" />
-        <child link="right_rear_wheel" />
-        <origin xyz="-0.25 0.2 0" rpy="0 0 0"/>
+        <child link="right_wheel" />
+        <origin xyz="${-((base_length/2.0)-0.05)} ${base_width/2.0} 0" rpy="0 0 0"/>
         <axis xyz="0 1 0"/>
     </joint>
@@ -141,5 +156,5 @@
         <parent link="base_link" />
         <child link="caster_wheel_link" />
-        <origin xyz="0.2 0 -0.05" rpy="0 0 0"/>
+        <origin xyz="0.2 0 ${-caster_wheel_radius}" rpy="0 0 0"/>
     </joint>
     <joint name="base_joint" type="fixed">

Commit message: working on my travel_bot...day_1

File: src/my_robot_description/urdf/mobile_base.xacro (robot description, xacro)
@@ -7,4 +7,11 @@
     <xacro:property name="wheel_length" value="0.1"/>
     <xacro:property name="caster_wheel_radius" value="0.1"/>
+    <xacro:property name="arm_base_length" value="0.1"/>
+    <xacro:property name="arm_base_width" value="0.1"/>
+    <xacro:property name="arm_base_height" value="0.02"/>
+    <xacro:property name="forearm_length" value="0.3"/>
+    <xacro:property name="forearm_radius" value="0.02"/>
+    <xacro:property name="hand_radius" value="0.02"/>
+    <xacro:property name="hand_lenght" value="0.3"/>
     <link name="base_link">
         <visual>
@@ -61,4 +68,52 @@
     <link name="base_footprint">
     </link>
+    <link name="arm_base_link">
+        <visual>
+            <geometry>
+                <box size="${arm_base_length} ${arm_base_width} ${arm_base_height}" />
+            </geometry>
+            <origin xyz="0 0 ${arm_base_height/2.0}" rpy="0 0 0" />
+            <material name="orange"/>
+        </visual>
+        <collision>
+            <geometry>
+                <box size="${arm_base_length} ${arm_base_width} ${arm_base_height}" />
+            </geometry>
+            <origin xyz="0 0 ${arm_base_height/2.0}" rpy="0 0 0" />
+        </collision>
+        <xacro:box_inertia m="0.5" x="${arm_base_length}" y="${arm_base_width}" z="${arm_base_height}" o_xyz="0 0 ${arm_base_height/2.0}" o_rpy="0 0 0" />
+    </link>
+    <link name="forearm_link">
+        <visual>
+            <geometry>
+                <cylinder radius="${forearm_radius}" length="${forearm_length}" />
+            </geometry>
+            <origin xyz="0 0 ${forearm_length/2.0}" rpy="0 0 0" />
+            <material name="yellow"/>
+        </visual>
+        <collision>
+                <geometry>
+                    <cylinder radius="${forearm_radius}" length="${forearm_length}"/>
+                </geometry>
+                <origin xyz="0 0 ${forearm_length/2.0}" rpy="0 0 0" />
+            </collision>
+            <xacro:cylinderical_inertia m="0.3" r="${forearm_radius}" l="${forearm_length}" o_xyz="0 0 ${forearm_length/2.0}" o_rpy="0 0 0" />
+    </link>
+    <link name="hand_link">
+        <visual>
+            <geometry>
+                <cylinder radius="${hand_radius}" length="${hand_lenght}"/>
+            </geometry>
+            <origin xyz="0 0 ${hand_lenght/2.0}" rpy="0 0 0"/>
+        </visual>
+        <material name="orange"/>
+        <collision>
+                <geometry>
+                    <cylinder radius="${hand_radius}" length="${hand_lenght}"/>
+                </geometry>
+                <origin xyz="0 0 ${hand_lenght/2.0}" rpy="0 0 0"/>
+            </collision>
+            <xacro:cylinderical_inertia m="0.3" r="${hand_radius}" l="${hand_lenght}" o_xyz="0 0 ${hand_lenght/2.0}" o_rpy="0 0 0" />
+    </link>
     <joint name="Base_left_r_wheel" type="continuous">
         <parent link="base_link" />
@@ -83,3 +138,24 @@
         <origin xyz="0 0 ${wheel_radius}" rpy="0 0 0"/>
     </joint>
+    <joint name="base_forearm_link" type="revolute">
+        <parent link="arm_base_link"/>
+        <child link="forearm_link"/>
+        <origin xyz="0 0 ${arm_base_height}" rpy="0 0 0"/>
+        <axis xyz="0 0 1"/>
+        <limit lower="0" upper="${pi/2.0}" effort="100" velocity="100"/>
+        <dynamics damping="0.3" friction="0.3"/>
+    </joint>
+    <joint name="hand_forearm_joint" type="revolute">
+        <parent link="forearm_link"/>
+        <child link="hand_link"/>
+        <origin xyz="0 0 ${forearm_length}" rpy="0 0 0"/>
+        <axis xyz="0 1 0"/>
+        <limit lower="0" upper="${pi/2.0}" effort="100" velocity="100"/>
+        <dynamics damping="0.3" friction="0.3"/>
+    </joint>
+    <joint name="base_arm_joint" type="fixed">
+        <parent link="base_link"/>
+        <child link="arm_base_link"/>
+        <origin xyz="0 0 ${base_height}" rpy="0 0 0"/>
+    </joint>
 </robot>

File: src/my_robot_description/urdf/mobile_base_gazebo.xacro (robot description, xacro)
@@ -18,4 +18,6 @@
                 <joint_name>Base_left_r_wheel</joint_name>
                 <joint_name>Base_right_r_wheel</joint_name>
+                <joint_name>base_forearm_link</joint_name>
+                <joint_name>hand_forearm_joint</joint_name>
         </plugin>
     </gazebo>

File: src/my_robot_description/urdf/robotic_arm_properties.xacro (robot description, xacro)
@@ -34,30 +34,3 @@
     </inertial>
     </xacro:macro>
-    <xacro:macro name="box_inertia" params="m x y z o_xyz o_rpy">
-    <inertial>
-        <origin xyz="${o_xyz}" rpy="${o_rpy}"/>
-        <mass value="${m}"/>
-        <inertia ixx="${m*(y*y + z*z)/12}" ixy="0" ixz="0"
-                 iyy="${m*(x*x + z*z)/12}" iyz="0"
-                 izz="${m*(y*y + x*x)/12}"/>
-    </inertial>
-    </xacro:macro>
-    <xacro:macro name="cylinderical_inertia" params="m r l o_xyz o_rpy">
-    <inertial>
-        <origin xyz="${o_xyz}" rpy="${o_rpy}"/>
-        <mass value="${m}"/>
-        <inertia ixx="${m*(3*r*r + l*l)/12}" ixy="0" ixz="0"
-                 iyy="${m*(3*r*r + l*l)/12}" iyz="0"
-                 izz="${m*(r*r)/2}"/>
-    </inertial>
-    </xacro:macro>
-    <xacro:macro name="spherical_inertia" params="m r  o_xyz o_rpy">
-    <inertial>
-        <origin xyz="${o_xyz}" rpy="${o_rpy}"/>
-        <mass value="${m}"/>
-        <inertia ixx="${m*(2*r*r)/3}" ixy="0" ixz="0"
-                 iyy="${m*(2*r*r)/3}" iyz="0"
-                 izz="${m*(r*r)/2}"/>
-    </inertial>
-    </xacro:macro>
 </robot>
